File: WTP/Circuit.sch (EAGLE design)
At the start: 13 parts, among them Q1 L78L06ABZ, Q2 16Mhz, U1 ATMEGA8-16PU, U2 +3.3v

Commit message: Updated schematics
Parts:
- added C8, C9: 0.1uF, resistor:C-EU050-025X075
- added R2: 10k, rcl:R-EU_VTA56
- added R3: (no value), ptc-ntc:NTC640
- added U$1: ESP01, esp8266modules:ESP01
Connections:
- net VCC renamed 12V
- new net N$10: R2.2, U1.PC1_(ADC1)
- new net N$6: B1.LV_RXO_1, U$1.TXD
- net 0: now also C8.2, C9.1, R3.1, U$1.GND, U1.GND_2
- net 3.3V: now also U$1.VCC
- net 5V: now also C9.2, U1.AREF
- net N$1: now also C8.1, U1.AVCC
- net N$8: now also B1.LV_TXI_1, U$1.RXD; no longer B1.LV_RXO_1
- net N$9: now also R2.1, R3.2, U1.PC0_(ADC0); no longer B1.LV_TXI_1
Other:
- moved on the sheet: B1, C1, C2, C3, C4, C5, C6, C7, Q1, Q2, R1, S1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
